File: PCB/servo_cpu/connectivity.kicad_sch (KiCad schematic)
At the start: 8 parts, among them J4 CONN, J7 USB_B_Micro, U10 SN65HVD232, U9 MAX485E

Commit message: cpu schematic
Connections:
- net Earth is gone; now on net GND: J4.SH
Changed lines of the file:
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@@
+    )
+  )
+  (symbol (lib_id "power:GND") (at 236.22 74.93 0) (unit 1)
+    (in_bom yes) (on_board yes) (dnp no)
+    (property "Reference" "#PWR03" (at 236.22 81.28 0)
+      (effects (font (size 1.27 1.27)) hide)
+    )
+    (property "Value" "GND" (at 240.03 78.74 0)
+      (effects (font (size 1.27 1.27)))
+    )
+    (property "Footprint" "" (at 236.22 74.93 0)
+      (effects (font (size 1.27 1.27)) hide)
+    )
+    (property "Datasheet" "" (at 236.22 74.93 0)
+      (effects (font (size 1.27 1.27)) hide)
+    )
+    (pin "1")
+    (instances
+      (project "servo_cpu"
+        (path "/db89e46c-646b-4fdd-b861-e9de706ced13/efadaaf3-3aa9-4d56-8b34-2b9a8a5957ea"
+          (reference "#PWR03") (unit 1)
+        )
+        (path "/db89e46c-646b-4fdd-b861-e9de706ced13/63791adc-fe14-4e15-9511-d81ede38744c"
+          (reference "#PWR080") (unit 1)
+        )
+      )
     )
   )
@@
         )
       )
-    )
-  )
-  (symbol (lib_id "power:Earth") (at 236.22 74.93 0) (unit 1)
-    (in_bom yes) (on_board yes) (dnp no) (fields_autoplaced)
-    (property "Reference" "#PWR068" (at 236.22 81.28 0)
-      (effects (font (size 1.27 1.27)) hide)
-    )
-    (property "Value" "Earth" (at 236.22 78.74 0)
-      (effects (font (size 1.27 1.27)) hide)
-    )
-    (property "Footprint" "" (at 236.22 74.93 0)
-      (effects (font (size 1.27 1.27)) hide)
-    )
-    (property "Datasheet" "~" (at 236.22 74.93 0)
-      (effects (font (size 1.27 1.27)) hide)
-    )
-    (pin "1")
-    (instances
-      (project "servo_cpu"
-        (path "/db89e46c-646b-4fdd-b861-e9de706ced13/bf198303-dc2c-4043-95ac-f79273257e19"
-          (reference "#PWR068") (unit 1)
-        )
-        (path "/db89e46c-646b-4fdd-b861-e9de706ced13/63791adc-fe14-4e15-9511-d81ede38744c"
-          (reference "#PWR080") (unit 1)
-        )
-      )

Commit message: cpu pcb
Connections:
- net +5V: now also J4.7
- no-connect marks 5 -> 4
Changed lines of the file:
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@@
   (junction (at 153.67 55.88) (diameter 0) (color 0 0 0 0)
   )
-  (no_connect (at 232.41 100.33))
   (no_connect (at 232.41 90.17))
   (no_connect (at 44.45 57.15))
@@
   )
   (wire (pts (xy 34.29 62.23) (xy 36.83 62.23))
+    (stroke (width 0) (type default))
+  )
+  (wire (pts (xy 227.33 100.33) (xy 232.41 100.33))
     (stroke (width 0) (type default))
   )
@@
         )
       )
+    )
+  )
+  (symbol (lib_id "power:+5V") (at 227.33 100.33 90) (unit 1)
+    (in_bom yes) (on_board yes) (dnp no) (fields_autoplaced)
+    (property "Reference" "#PWR049" (at 231.14 100.33 0)
+      (effects (font (size 1.27 1.27)) hide)
+    )
+    (property "Value" "+5V" (at 223.52 100.965 90)
+      (effects (font (size 1.27 1.27)) (justify left))
+    )
+    (property "Footprint" "" (at 227.33 100.33 0)
+      (effects (font (size 1.27 1.27)) hide)
+    )
+    (property "Datasheet" "" (at 227.33 100.33 0)
+      (effects (font (size 1.27 1.27)) hide)
+    )
+    (pin "1")
+    (instances
+      (project "servo_cpu"
+        (path "/db89e46c-646b-4fdd-b861-e9de706ced13/731cc340-9654-433e-bcf1-701f3d0fb633"
+          (reference "#PWR049") (unit 1)
+        )
+        (path "/db89e46c-646b-4fdd-b861-e9de706ced13/63791adc-fe14-4e15-9511-d81ede38744c"
+          (reference "#PWR068") (unit 1)
+        )
+      )

Commit message: CPU schematic done
Parts:
- added J9: EXT, Connector_PinHeader_2.54mm:PinHeader_2x04_P2.54mm_Horizontal, symbol Connector_Generic:Conn_02x04_Odd_Even
Connections:
- net +5V: now also J9.1 (Pin_1)
- net GND: now also J9.2 (Pin_2)
- new net EXT_CLK: J9.4 (Pin_4)
- new net EXT_CS: J9.7 (Pin_7)
- new net EXT_INT: J9.3 (Pin_3)
- new net EXT_MISO: J9.6 (Pin_6)
- new net EXT_MOSI: J9.8 (Pin_8)
- new net EXT_RESET: J9.5 (Pin_5)
Other:
- note added: "CAN transciever"
- note added: "Extension port"
- note added: "RS485 transciever"
- note added: "USB port"
- title: (none) -> Fieldbus intrefaces
Changed lines of the file:
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@@
 (kicad_sch (version 20230121) (generator eeschema)
   (paper "A4")
+  (title_block
+    (title "Fieldbus intrefaces")
+    (date "2023-03-06")
+    (rev "1")
+    (comment 1 "W. Burdecki 2023")
+    (comment 2 "github.com/wiciu15")
+  )
   (junction (at 34.29 62.23) (diameter 0) (color 0 0 0 0)
   )
@@
     (stroke (width 0) (type default))
   )
+  (text "USB port" (at 31.75 35.56 0)
+    (effects (font (size 3 3)) (justify left bottom))
+  )
+  (text "Extension port" (at 40.64 101.6 0)
+    (effects (font (size 3 3)) (justify left bottom))
+  )
+  (text "RS485 transciever" (at 123.19 19.05 0)
+    (effects (font (size 3 3)) (justify left bottom))
+  )
+  (text "CAN transciever" (at 137.16 97.79 0)
+    (effects (font (size 3 3)) (justify left bottom))
+  )
   (global_label "MODBUS_TX" (shape input) (at 127 55.88 180) (fields_autoplaced)
     (effects (font (size 1.27 1.27)) (justify right))
@@
     )
   )
+  (global_label "EXT_MISO" (shape input) (at 59.69 115.57 0) (fields_autoplaced)
+    (effects (font (size 1.27 1.27)) (justify left))
+    (property "Intersheetrefs" "${INTERSHEET_REFS}" (at 71.4857 115.57 0)
+      (effects (font (size 1.27 1.27)) (justify left) hide)
+    )
+  )
   (global_label "B-" (shape input) (at 232.41 87.63 180) (fields_autoplaced)
     (effects (font (size 1.27 1.27)) (justify right))
@@
     )
   )
+  (global_label "EXT_CLK" (shape input) (at 59.69 113.03 0) (fields_autoplaced)
+    (effects (font (size 1.27 1.27)) (justify left))
+    (property "Intersheetrefs" "${INTERSHEET_REFS}" (at 70.4576 113.03 0)
+      (effects (font (size 1.27 1.27)) (justify left) hide)
+    )
+  )
   (global_label "USB_P" (shape input) (at 50.8 52.07 0) (fields_autoplaced)
     (effects (font (size 1.27 1.27)) (justify left))
@@
     )
   )
+  (global_label "EXT_CS" (shape input) (at 46.99 118.11 180) (fields_autoplaced)
+    (effects (font (size 1.27 1.27)) (justify right))
+    (property "Intersheetrefs" "${INTERSHEET_REFS}" (at 37.311 118.11 0)
+      (effects (font (size 1.27 1.27)) (justify right) hide)
+    )
+  )
   (global_label "USB_N" (shape input) (at 50.8 54.61 0) (fields_autoplaced)
     (effects (font (size 1.27 1.27)) (justify left))
@@
     )
   )
+  (global_label "EXT_MOSI" (shape input) (at 59.69 118.11 0) (fields_autoplaced)
+    (effects (font (size 1.27 1.27)) (justify left))
+    (property "Intersheetrefs" "${INTERSHEET_REFS}" (at 71.4857 118.11 0)
+      (effects (font (size 1.27 1.27)) (justify left) hide)
+    )
+  )
   (global_label "CAN_TX" (shape input) (at 144.78 121.92 180) (fields_autoplaced)
     (effects (font (size 1.27 1.27)) (justify right))
@@
     )
   )
+  (global_label "EXT_RESET" (shape input) (at 46.99 115.57 180) (fields_autoplaced)
+    (effects (font (size 1.27 1.27)) (justify right))
+    (property "Intersheetrefs" "${INTERSHEET_REFS}" (at 34.0454 115.57 0)
+      (effects (font (size 1.27 1.27)) (justify right) hide)
+    )
+  )
+  (global_label "EXT_INT" (shape input) (at 46.99 113.03 180) (fields_autoplaced)
+    (effects (font (size 1.27 1.27)) (justify right))
+    (property "Intersheetrefs" "${INTERSHEET_REFS}" (at 36.8876 113.03 0)
+      (effects (font (size 1.27 1.27)) (justify right) hide)
+    )
+  )
   (global_label "CANL" (shape input) (at 232.41 95.25 180) (fields_autoplaced)
     (effects (font (size 1.27 1.27)) (justify right))
@@
         (path "/db89e46c-646b-4fdd-b861-e9de706ced13/63791adc-fe14-4e15-9511-d81ede38744c"
           (reference "D3") (unit 1)
+        )
+      )
+    )
+  )
+  (symbol (lib_id "power:+5V") (at 46.99 110.49 90) (unit 1)
+    (in_bom yes) (on_board yes) (dnp no)
+    (property "Reference" "#PWR049" (at 50.8 110.49 0)
+      (effects (font (size 1.27 1.27)) hide)
+    )
+    (property "Value" "+5V" (at 43.18 110.49 90)
+      (effects (font (size 1.27 1.27)) (justify left))
+    )
+    (property "Footprint" "" (at 46.99 110.49 0)
+      (effects (font (size 1.27 1.27)) hide)
+    )
+    (property "Datasheet" "" (at 46.99 110.49 0)
+      (effects (font (size 1.27 1.27)) hide)
+    )
+    (pin "1")
+    (instances
+      (project "servo_cpu"
+        (path "/db89e46c-646b-4fdd-b861-e9de706ced13/731cc340-9654-433e-bcf1-701f3d0fb633"
+          (reference "#PWR049") (unit 1)
+        )
+        (path "/db89e46c-646b-4fdd-b861-e9de706ced13/63791adc-fe14-4e15-9511-d81ede38744c"
+          (reference "#PWR0138") (unit 1)
         )
       )
@@
     )
   )
+  (symbol (lib_id "power:GND") (at 59.69 110.49 90) (unit 1)
+    (in_bom yes) (on_board yes) (dnp no)
+    (property "Reference" "#PWR03" (at 66.04 110.49 0)
+      (effects (font (size 1.27 1.27)) hide)
+    )
+    (property "Value" "GND" (at 63.5 106.68 0)
+      (effects (font (size 1.27 1.27)))
+    )
+    (property "Footprint" "" (at 59.69 110.49 0)
+      (effects (font (size 1.27 1.27)) hide)
+    )
+    (property "Datasheet" "" (at 59.69 110.49 0)
+      (effects (font (size 1.27 1.27)) hide)
+    )
+    (pin "1")
+    (instances
+      (project "servo_cpu"
+        (path "/db89e46c-646b-4fdd-b861-e9de706ced13/efadaaf3-3aa9-4d56-8b34-2b9a8a5957ea"
+          (reference "#PWR03") (unit 1)
+        )
+        (path "/db89e46c-646b-4fdd-b861-e9de706ced13/63791adc-fe14-4e15-9511-d81ede38744c"
+          (reference "#PWR0139") (unit 1)
+        )
+      )
+    )
+  )
   (symbol (lib_id "power:GND") (at 139.7 113.03 0) (unit 1)
     (in_bom yes) (on_board yes) (dnp no)
@@
         )
       )
+    )
+  )
+  (symbol (lib_id "Connector_Generic:Conn_02x04_Odd_Even") (at 52.07 113.03 0) (unit 1)
+    (in_bom yes) (on_board yes) (dnp no) (fields_autoplaced)
+    (property "Reference" "J9" (at 53.34 105.41 0)
+      (effects (font (size 1.27 1.27)))
+    )
+    (property "Value" "EXT" (at 53.34 107.95 0)
+      (effects (font (size 1.27 1.27)))
+    )
+    (property "Footprint" "Connector_PinHeader_2.54mm:PinHeader_2x04_P2.54mm_Horizontal" (at 52.07 113.03 0)
+      (effects (font (size 1.27 1.27)) hide)
+    )
+    (property "Datasheet" "~" (at 52.07 113.03 0)
+      (effects (font (size 1.27 1.27)) hide)
+    )
+    (pin "1")
+    (pin "2")
+    (pin "3")
+    (pin "4")
+    (pin "5")
+    (pin "6")
+    (pin "7")
+    (pin "8")
+    (instances
+      (project "servo_cpu"
+        (path "/db89e46c-646b-4fdd-b861-e9de706ced13/63791adc-fe14-4e15-9511-d81ede38744c"
+          (reference "J9") (unit 1)
+        )
+      )

Commit message: cpu pcb
Parts:
- added R54: 470R, symbol Device:R_Small
- added R56: 1k, symbol Device:R_Small
Connections:
- net +5V: now also R56.1
- net A+: now also R54.1
- net B-: now also R56.2
- net GND: now also R54.2
Other:
- moved on the sheet: D3, D4
Changed lines of the file:
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@@
   (junction (at 34.29 62.23) (diameter 0) (color 0 0 0 0)
   )
+  (junction (at 158.75 48.26) (diameter 0) (color 0 0 0 0)
+  )
   (junction (at 137.16 27.94) (diameter 0) (color 0 0 0 0)
   )
   (junction (at 168.91 48.26) (diameter 0) (color 0 0 0 0)
   )
-  (junction (at 161.29 67.31) (diameter 0) (color 0 0 0 0)
+  (junction (at 161.29 73.66) (diameter 0) (color 0 0 0 0)
   )
   (junction (at 139.7 107.95) (diameter 0) (color 0 0 0 0)
+  )
+  (junction (at 158.75 55.88) (diameter 0) (color 0 0 0 0)
   )
   (junction (at 153.67 55.88) (diameter 0) (color 0 0 0 0)
@@
   (no_connect (at 44.45 46.99))
   (no_connect (at 232.41 97.79))
-  (wire (pts (xy 153.67 67.31) (xy 161.29 67.31))
+  (wire (pts (xy 153.67 73.66) (xy 161.29 73.66))
     (stroke (width 0) (type default))
   )
@@
     (stroke (width 0) (type default))
   )
+  (wire (pts (xy 158.75 55.88) (xy 173.99 55.88))
+    (stroke (width 0) (type default))
+  )
   (wire (pts (xy 227.33 100.33) (xy 232.41 100.33))
     (stroke (width 0) (type default))
@@
     (stroke (width 0) (type default))
   )
-  (wire (pts (xy 153.67 55.88) (xy 173.99 55.88))
+  (wire (pts (xy 153.67 55.88) (xy 158.75 55.88))
     (stroke (width 0) (type default))
   )
@@
     (stroke (width 0) (type default))
   )
+  (wire (pts (xy 158.75 48.26) (xy 168.91 48.26))
+    (stroke (width 0) (type default))
+  )
   (wire (pts (xy 228.6 102.87) (xy 232.41 102.87))
     (stroke (width 0) (type default))
@@
     (stroke (width 0) (type default))
   )
-  (wire (pts (xy 161.29 67.31) (xy 168.91 67.31))
+  (wire (pts (xy 161.29 73.66) (xy 168.91 73.66))
     (stroke (width 0) (type default))
   )
@@
     (stroke (width 0) (type default))
   )
-  (wire (pts (xy 153.67 55.88) (xy 153.67 59.69))
-    (stroke (width 0) (type default))
-  )
-  (wire (pts (xy 168.91 48.26) (xy 168.91 59.69))
+  (wire (pts (xy 153.67 55.88) (xy 153.67 66.04))
+    (stroke (width 0) (type default))
+  )
+  (wire (pts (xy 168.91 48.26) (xy 168.91 66.04))
     (stroke (width 0) (type default))
   )
@@
     (stroke (width 0) (type default))
   )
-  (wire (pts (xy 147.32 48.26) (xy 168.91 48.26))
+  (wire (pts (xy 147.32 48.26) (xy 158.75 48.26))
     (stroke (width 0) (type default))
   )
@@
     )
   )
-  (symbol (lib_id "Diode:BZT52Bxx") (at 168.91 63.5 270) (unit 1)
-    (in_bom yes) (on_board yes) (dnp no) (fields_autoplaced)
-    (property "Reference" "D4" (at 171.45 62.865 90)
-      (effects (font (size 1.27 1.27)) (justify left))
-    )
-    (property "Value" "BZT52B6v2" (at 171.45 65.405 90)
-      (effects (font (size 1.27 1.27)) (justify left))
-    )
-    (property "Footprint" "Diode_SMD:D_SOD-123F" (at 164.465 63.5 0)
-      (effects (font (size 1.27 1.27)) hide)
-    )
-    (property "Datasheet" "https://diotec.com/tl_files/diotec/files/pdf/datasheets/bzt52b2v4.pdf" (at 168.91 63.5 0)
+  (symbol (lib_id "Diode:BZT52Bxx") (at 168.91 69.85 270) (unit 1)
+    (in_bom yes) (on_board yes) (dnp no) (fields_autoplaced)
+    (property "Reference" "D4" (at 171.45 69.215 90)
+      (effects (font (size 1.27 1.27)) (justify left))
+    )
+    (property "Value" "BZT52B6v2" (at 171.45 71.755 90)
+      (effects (font (size 1.27 1.27)) (justify left))
+    )
+    (property "Footprint" "Diode_SMD:D_SOD-123F" (at 164.465 69.85 0)
+      (effects (font (size 1.27 1.27)) hide)
+    )
+    (property "Datasheet" "https://diotec.com/tl_files/diotec/files/pdf/datasheets/bzt52b2v4.pdf" (at 168.91 69.85 0)
       (effects (font (size 1.27 1.27)) hide)
     )
@@
     )
   )
-  (symbol (lib_id "Diode:BZT52Bxx") (at 153.67 63.5 270) (unit 1)
-    (in_bom yes) (on_board yes) (dnp no) (fields_autoplaced)
-    (property "Reference" "D3" (at 156.21 62.865 90)
-      (effects (font (size 1.27 1.27)) (justify left))
-    )
-    (property "Value" "BZT52B6v2" (at 156.21 65.405 90)
-      (effects (font (size 1.27 1.27)) (justify left))
-    )
-    (property "Footprint" "Diode_SMD:D_SOD-123F" (at 149.225 63.5 0)
-      (effects (font (size 1.27 1.27)) hide)
-    )
-    (property "Datasheet" "https://diotec.com/tl_files/diotec/files/pdf/datasheets/bzt52b2v4.pdf" (at 153.67 63.5 0)
+  (symbol (lib_id "Diode:BZT52Bxx") (at 153.67 69.85 270) (unit 1)
+    (in_bom yes) (on_board yes) (dnp no) (fields_autoplaced)
+    (property "Reference" "D3" (at 156.21 69.215 90)
+      (effects (font (size 1.27 1.27)) (justify left))
+    )
+    (property "Value" "BZT52B6v2" (at 156.21 71.755 90)
+      (effects (font (size 1.27 1.27)) (justify left))
+    )
+    (property "Footprint" "Diode_SMD:D_SOD-123F" (at 149.225 69.85 0)
+      (effects (font (size 1.27 1.27)) hide)
+    )
+    (property "Datasheet" "https://diotec.com/tl_files/diotec/files/pdf/datasheets/bzt52b2v4.pdf" (at 153.67 69.85 0)
       (effects (font (size 1.27 1.27)) hide)
     )
@@
     )
   )
+  (symbol (lib_id "power:GND") (at 158.75 60.96 0) (unit 1)
+    (in_bom yes) (on_board yes) (dnp no)
+    (property "Reference" "#PWR03" (at 158.75 67.31 0)
+      (effects (font (size 1.27 1.27)) hide)
+    )
+    (property "Value" "GND" (at 162.56 64.77 0)
+      (effects (font (size 1.27 1.27)))
+    )
+    (property "Footprint" "" (at 158.75 60.96 0)
+      (effects (font (size 1.27 1.27)) hide)
+    )
+    (property "Datasheet" "" (at 158.75 60.96 0)
+      (effects (font (size 1.27 1.27)) hide)
+    )
+    (pin "1")
+    (instances
+      (project "servo_cpu"
+        (path "/db89e46c-646b-4fdd-b861-e9de706ced13/efadaaf3-3aa9-4d56-8b34-2b9a8a5957ea"
+          (reference "#PWR03") (unit 1)
+        )
+        (path "/db89e46c-646b-4fdd-b861-e9de706ced13"
+          (reference "#PWR022") (unit 1)
+        )
+        (path "/db89e46c-646b-4fdd-b861-e9de706ced13/731cc340-9654-433e-bcf1-701f3d0fb633"
+          (reference "#PWR041") (unit 1)
+        )
+        (path "/db89e46c-646b-4fdd-b861-e9de706ced13/63791adc-fe14-4e15-9511-d81ede38744c"
+          (reference "#PWR0149") (unit 1)
+        )
+      )
+    )
+  )
+  (symbol (lib_id "power:+5V") (at 158.75 43.18 0) (unit 1)
+    (in_bom yes) (on_board yes) (dnp no) (fields_autoplaced)
+    (property "Reference" "#PWR049" (at 158.75 46.99 0)
+      (effects (font (size 1.27 1.27)) hide)
+    )
+    (property "Value" "+5V" (at 158.75 39.37 0)
+      (effects (font (size 1.27 1.27)))
+    )
+    (property "Footprint" "" (at 158.75 43.18 0)
+      (effects (font (size 1.27 1.27)) hide)
+    )
+    (property "Datasheet" "" (at 158.75 43.18 0)
+      (effects (font (size 1.27 1.27)) hide)
+    )
+    (pin "1")
+    (instances
+      (project "servo_cpu"
+        (path "/db89e46c-646b-4fdd-b861-e9de706ced13/731cc340-9654-433e-bcf1-701f3d0fb633"
+          (reference "#PWR049") (unit 1)
+        )
+        (path "/db89e46c-646b-4fdd-b861-e9de706ced13/63791adc-fe14-4e15-9511-d81ede38744c"
+          (reference "#PWR0148") (unit 1)
+        )
+      )
+    )
+  )
   (symbol (lib_id "Connector:USB_B_Micro") (at 36.83 52.07 0) (unit 1)
     (in_bom yes) (on_board yes) (dnp no) (fields_autoplaced)
@@
     )
   )
-  (symbol (lib_id "power:GND") (at 161.29 67.31 0) (unit 1)
-    (in_bom yes) (on_board yes) (dnp no)
-    (property "Reference" "#PWR03" (at 161.29 73.66 0)
-      (effects (font (size 1.27 1.27)) hide)
-    )
-    (property "Value" "GND" (at 165.1 71.12 0)
-      (effects (font (size 1.27 1.27)))
-    )
-    (property "Footprint" "" (at 161.29 67.31 0)
-      (effects (font (size 1.27 1.27)) hide)
-    )
-    (property "Datasheet" "" (at 161.29 67.31 0)
+  (symbol (lib_id "power:GND") (at 161.29 73.66 0) (unit 1)
+    (in_bom yes) (on_board yes) (dnp no)
+    (property "Reference" "#PWR03" (at 161.29 80.01 0)
+      (effects (font (size 1.27 1.27)) hide)
+    )
+    (property "Value" "GND" (at 165.1 77.47 0)
+      (effects (font (size 1.27 1.27)))
+    )
+    (property "Footprint" "" (at 161.29 73.66 0)
+      (effects (font (size 1.27 1.27)) hide)
+    )
+    (property "Datasheet" "" (at 161.29 73.66 0)
       (effects (font (size 1.27 1.27)) hide)
     )
@@
     )
   )
+  (symbol (lib_id "Device:R_Small") (at 158.75 45.72 0) (unit 1)
+    (in_bom yes) (on_board yes) (dnp no)
+    (property "Reference" "R56" (at 161.29 45.085 0)
+      (effects (font (size 1.27 1.27)) (justify left))
+    )
+    (property "Value" "1k" (at 161.29 46.99 0)
+      (effects (font (size 1.27 1.27)) (justify left))
+    )
+    (property "Footprint" "" (at 158.75 45.72 0)
+      (effects (font (size 1.27 1.27)) hide)
+    )
+    (property "Datasheet" "~" (at 158.75 45.72 0)
+      (effects (font (size 1.27 1.27)) hide)
+    )
+    (pin "1")
+    (pin "2")
+    (instances
+      (project "servo_cpu"
+        (path "/db89e46c-646b-4fdd-b861-e9de706ced13/bf198303-dc2c-4043-95ac-f79273257e19"
+          (reference "R56") (unit 1)
+        )
+        (path "/db89e46c-646b-4fdd-b861-e9de706ced13/63791adc-fe14-4e15-9511-d81ede38744c"
+          (reference "R55") (unit 1)
+        )
+      )
+    )
+  )
   (symbol (lib_id "Interface_CAN_LIN:SN65HVD232") (at 154.94 124.46 0) (unit 1)
     (in_bom yes) (on_board yes) (dnp no) (fields_autoplaced)
@@
         )
       )
+    )
+  )
+  (symbol (lib_id "Device:R_Small") (at 158.75 58.42 0) (unit 1)
+    (in_bom yes) (on_board yes) (dnp no)
+    (property "Reference" "R54" (at 161.29 57.785 0)
+      (effects (font (size 1.27 1.27)) (justify left))
+    )
+    (property "Value" "470R" (at 161.29 59.69 0)
+      (effects (font (size 1.27 1.27)) (justify left))
+    )
+    (property "Footprint" "" (at 158.75 58.42 0)
+      (effects (font (size 1.27 1.27)) hide)
+    )
+    (property "Datasheet" "~" (at 158.75 58.42 0)
+      (effects (font (size 1.27 1.27)) hide)
+    )
+    (pin "1")
+    (pin "2")
+    (instances
+      (project "servo_cpu"
+        (path "/db89e46c-646b-4fdd-b861-e9de706ced13/bf198303-dc2c-4043-95ac-f79273257e19"
+          (reference "R54") (unit 1)
+        )
+        (path "/db89e46c-646b-4fdd-b861-e9de706ced13/63791adc-fe14-4e15-9511-d81ede38744c"
+          (reference "R58") (unit 1)
+        )
+      )
