File: PCB/servo_cpu/connectivity.kicad_sch (KiCad schematic)
At the start: 11 parts, among them J4 CONN, J7 USB_B_Micro, J9 EXT, U10 SN65HVD232, U9 MAX485E

Commit message: cpu pcb layout
Parts:
- removed J7: USB_B_Micro, Connector_USB:USB_Mini-B_Wuerth_65100516121_Horizontal, symbol Connector:USB_B_Micro
- added J7: USB_B, USB_B_JST_Vertical:USB, symbol Connector:USB_B
- C1, C2: footprint (none) -> Capacitor_SMD:C_0805_2012Metric_Pad1.18x1.45mm_HandSolder
- R54, R56: footprint (none) -> Resistor_SMD:R_0805_2012Metric_Pad1.20x1.40mm_HandSolder
- U9: footprint (none) -> Package_SO:SO-8_3.9x4.9mm_P1.27mm
Connections:
- net GND: now also J7.4 (GND), J7.5 (Shield)
- net USB_N: now also J7.2 (D-)
- net USB_P: now also J7.3 (D+)
- no-connect marks 4 -> 3
Changed lines of the file:
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@@
     (comment 2 "github.com/wiciu15")
   )
+  (junction (at 158.75 48.26) (diameter 0) (color 0 0 0 0)
+  )
+  (junction (at 137.16 27.94) (diameter 0) (color 0 0 0 0)
+  )
+  (junction (at 168.91 48.26) (diameter 0) (color 0 0 0 0)
+  )
+  (junction (at 161.29 73.66) (diameter 0) (color 0 0 0 0)
+  )
+  (junction (at 139.7 107.95) (diameter 0) (color 0 0 0 0)
+  )
+  (junction (at 158.75 55.88) (diameter 0) (color 0 0 0 0)
+  )
   (junction (at 34.29 62.23) (diameter 0) (color 0 0 0 0)
   )
-  (junction (at 158.75 48.26) (diameter 0) (color 0 0 0 0)
-  )
-  (junction (at 137.16 27.94) (diameter 0) (color 0 0 0 0)
-  )
-  (junction (at 168.91 48.26) (diameter 0) (color 0 0 0 0)
-  )
-  (junction (at 161.29 73.66) (diameter 0) (color 0 0 0 0)
-  )
-  (junction (at 139.7 107.95) (diameter 0) (color 0 0 0 0)
-  )
-  (junction (at 158.75 55.88) (diameter 0) (color 0 0 0 0)
-  )
   (junction (at 153.67 55.88) (diameter 0) (color 0 0 0 0)
   )
   (no_connect (at 232.41 90.17))
-  (no_connect (at 44.45 57.15))
   (no_connect (at 44.45 46.99))
   (no_connect (at 232.41 97.79))
@@
       (effects (font (size 1.27 1.27)) (justify left))
     )
-    (property "Footprint" "" (at 137.16 68.58 0)
+    (property "Footprint" "Package_SO:SO-8_3.9x4.9mm_P1.27mm" (at 137.16 68.58 0)
       (effects (font (size 1.27 1.27)) hide)
     )
@@
     )
   )
-  (symbol (lib_id "power:+5V") (at 158.75 43.18 0) (unit 1)
-    (in_bom yes) (on_board yes) (dnp no) (fields_autoplaced)
-    (property "Reference" "#PWR049" (at 158.75 46.99 0)
-      (effects (font (size 1.27 1.27)) hide)
-    )
-    (property "Value" "+5V" (at 158.75 39.37 0)
-      (effects (font (size 1.27 1.27)))
-    )
-    (property "Footprint" "" (at 158.75 43.18 0)
-      (effects (font (size 1.27 1.27)) hide)
-    )
-    (property "Datasheet" "" (at 158.75 43.18 0)
-      (effects (font (size 1.27 1.27)) hide)
-    )
-    (pin "1")
-    (instances
-      (project "servo_cpu"
-        (path "/db89e46c-646b-4fdd-b861-e9de706ced13/731cc340-9654-433e-bcf1-701f3d0fb633"
-          (reference "#PWR049") (unit 1)
-        )
-        (path "/db89e46c-646b-4fdd-b861-e9de706ced13/63791adc-fe14-4e15-9511-d81ede38744c"
-          (reference "#PWR0148") (unit 1)
-        )
-      )
-    )
-  )
-  (symbol (lib_id "Connector:USB_B_Micro") (at 36.83 52.07 0) (unit 1)
+  (symbol (lib_id "Connector:USB_B") (at 36.83 52.07 0) (unit 1)
     (in_bom yes) (on_board yes) (dnp no) (fields_autoplaced)
     (property "Reference" "J7" (at 36.83 40.64 0)
       (effects (font (size 1.27 1.27)))
     )
-    (property "Value" "USB_B_Micro" (at 36.83 43.18 0)
-      (effects (font (size 1.27 1.27)))
-    )
-    (property "Footprint" "Connector_USB:USB_Mini-B_Wuerth_65100516121_Horizontal" (at 40.64 53.34 0)
-      (effects (font (size 1.27 1.27)) hide)
-    )
-    (property "Datasheet" "~" (at 40.64 53.34 0)
+    (property "Value" "USB_B" (at 36.83 43.18 0)
+      (effects (font (size 1.27 1.27)))
+    )
+    (property "Footprint" "USB_B_JST_Vertical:USB" (at 40.64 53.34 0)
+      (effects (font (size 1.27 1.27)) hide)
+    )
+    (property "Datasheet" " ~" (at 40.64 53.34 0)
       (effects (font (size 1.27 1.27)) hide)
     )
@@
     (pin "4")
     (pin "5")
-    (pin "6")
     (instances
       (project "servo_cpu"
         (path "/db89e46c-646b-4fdd-b861-e9de706ced13/63791adc-fe14-4e15-9511-d81ede38744c"
           (reference "J7") (unit 1)
+        )
+      )
+    )
+  )
+  (symbol (lib_id "power:+5V") (at 158.75 43.18 0) (unit 1)
+    (in_bom yes) (on_board yes) (dnp no) (fields_autoplaced)
+    (property "Reference" "#PWR049" (at 158.75 46.99 0)
+      (effects (font (size 1.27 1.27)) hide)
+    )
+    (property "Value" "+5V" (at 158.75 39.37 0)
+      (effects (font (size 1.27 1.27)))
+    )
+    (property "Footprint" "" (at 158.75 43.18 0)
+      (effects (font (size 1.27 1.27)) hide)
+    )
+    (property "Datasheet" "" (at 158.75 43.18 0)
+      (effects (font (size 1.27 1.27)) hide)
+    )
+    (pin "1")
+    (instances
+      (project "servo_cpu"
+        (path "/db89e46c-646b-4fdd-b861-e9de706ced13/731cc340-9654-433e-bcf1-701f3d0fb633"
+          (reference "#PWR049") (unit 1)
+        )
+        (path "/db89e46c-646b-4fdd-b861-e9de706ced13/63791adc-fe14-4e15-9511-d81ede38744c"
+          (reference "#PWR0148") (unit 1)
         )
       )
@@
       (effects (font (size 1.27 1.27)) (justify left))
     )
-    (property "Footprint" "" (at 158.75 45.72 0)
+    (property "Footprint" "Resistor_SMD:R_0805_2012Metric_Pad1.20x1.40mm_HandSolder" (at 158.75 45.72 0)
       (effects (font (size 1.27 1.27)) hide)
     )
@@
       (effects (font (size 1.27 1.27)) (justify left))
     )
-    (property "Footprint" "" (at 139.7 110.49 0)
+    (property "Footprint" "Capacitor_SMD:C_0805_2012Metric_Pad1.18x1.45mm_HandSolder" (at 139.7 110.49 0)
       (effects (font (size 1.27 1.27)) hide)
     )
@@
       (effects (font (size 1.27 1.27)) (justify left))
     )
-    (property "Footprint" "" (at 158.75 58.42 0)
+    (property "Footprint" "Resistor_SMD:R_0805_2012Metric_Pad1.20x1.40mm_HandSolder" (at 158.75 58.42 0)
       (effects (font (size 1.27 1.27)) hide)
     )
@@
       (effects (font (size 1.27 1.27)) (justify left))
     )
-    (property "Footprint" "" (at 125.73 30.48 0)
-      (effects (font (size 1.27 1.27)) hide)
-    )
+    (property "Footprint" "Capacitor_SMD:C_0805_2012Metric_Pad1.18x1.45mm_HandSolder" (at 125.73 30.48 0)
+      (effects (font (size 1.27 1.27)) hide)
+    )
