File: PCB/servo_cpu/display.kicad_sch (KiCad schematic)
At the start: 7 parts

Commit message: cpu pcb
Parts:
- added D5, D6: LED, symbol Device:LED
- added R15, R16: 1k, symbol Device:R_Small
- added SW1: ENTER, Button_Switch_SMD:SW_SPST_B3S-1000, symbol Switch:SW_Push
- added SW2: ESC, Button_Switch_SMD:SW_SPST_B3S-1000, symbol Switch:SW_Push
- added SW3: UP, Button_Switch_SMD:SW_SPST_B3S-1000, symbol Switch:SW_Push
- added SW4: DOWN, Button_Switch_SMD:SW_SPST_B3S-1000, symbol Switch:SW_Push
Connections:
- net GND: now also D5.1 (K), D6.1 (K), SW1.2, SW2.2, SW3.2, SW4.2
- new net: D6.2 (A), R16.2
- new net: D5.2 (A), R15.2
- new net BTN_DOWN: SW4.1
- new net BTN_ENTER: SW1.1
- new net BTN_ESC: SW2.1
- new net BTN_UP: SW3.1
- new net LED_ERROR: R16.1
- new net LED_STATUS: R15.1
Other:
- moved on the sheet: C1, C2, C3, C4, C5, DS1, R1

Commit message: cpu schematic
Parts:
- D5: value LED -> GREEN_LED; footprint (none) -> Diode_SMD:D_1206_3216Metric_Pad1.42x1.75mm_HandSolder
- D6: value LED -> RED_LED; footprint (none) -> Diode_SMD:D_1206_3216Metric_Pad1.42x1.75mm_HandSolder
Changed lines of the file:
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@@
       (effects (font (size 1.27 1.27)) (justify right))
     )
-    (property "Value" "LED" (at 132.08 135.5725 90)
+    (property "Value" "RED_LED" (at 132.08 135.5725 90)
       (effects (font (size 1.27 1.27)) (justify right))
     )
-    (property "Footprint" "" (at 128.27 132.08 0)
+    (property "Footprint" "Diode_SMD:D_1206_3216Metric_Pad1.42x1.75mm_HandSolder" (at 128.27 132.08 0)
       (effects (font (size 1.27 1.27)) hide)
     )
@@
       (effects (font (size 1.27 1.27)) (justify right))
     )
-    (property "Value" "LED" (at 132.08 108.9025 90)
+    (property "Value" "GREEN_LED" (at 132.08 108.9025 90)
       (effects (font (size 1.27 1.27)) (justify right))
     )
-    (property "Footprint" "" (at 128.27 105.41 0)
+    (property "Footprint" "Diode_SMD:D_1206_3216Metric_Pad1.42x1.75mm_HandSolder" (at 128.27 105.41 0)
       (effects (font (size 1.27 1.27)) hide)
     )

Commit message: CPU schematic done
Parts:
- added C48, C49, C50, C51: 100n, symbol Device:C_Small
Connections:
- net BTN_DOWN: now also C51.1
- net BTN_ENTER: now also C48.1
- net BTN_ESC: now also C49.1
- net BTN_UP: now also C50.1
- net GND: now also C48.2, C49.2, C50.2, C51.2
Other:
- note added: "1,3 inch OLED display"
- note added: "Buttons"
- note added: "Status LED"
- title: (none) -> Display
- moved on the sheet: D5, D6, R15, R16, SW1, SW2, SW4

Commit message: cpu pcb layout
Parts:
- C1, C2, C3, C4, C48, C49, C5, C50, C51: footprint (none) -> Capacitor_SMD:C_0805_2012Metric_Pad1.18x1.45mm_HandSolder
- R1, R15, R16: footprint (none) -> Resistor_SMD:R_0805_2012Metric_Pad1.20x1.40mm_HandSolder
Changed lines of the file:
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@@
       (effects (font (size 1.27 1.27)) (justify left))
     )
-    (property "Footprint" "" (at 134.62 86.36 0)
+    (property "Footprint" "Capacitor_SMD:C_0805_2012Metric_Pad1.18x1.45mm_HandSolder" (at 134.62 86.36 0)
       (effects (font (size 1.27 1.27)) hide)
     )
@@
       (effects (font (size 1.27 1.27)) (justify left))
     )
-    (property "Footprint" "" (at 134.62 35.56 0)
+    (property "Footprint" "Capacitor_SMD:C_0805_2012Metric_Pad1.18x1.45mm_HandSolder" (at 134.62 35.56 0)
       (effects (font (size 1.27 1.27)) hide)
     )
@@
       (effects (font (size 1.27 1.27)) (justify left))
     )
-    (property "Footprint" "" (at 41.91 60.96 0)
+    (property "Footprint" "Capacitor_SMD:C_0805_2012Metric_Pad1.18x1.45mm_HandSolder" (at 41.91 60.96 0)
       (effects (font (size 1.27 1.27)) hide)
     )
@@
       (effects (font (size 1.27 1.27)) (justify left))
     )
-    (property "Footprint" "" (at 134.62 69.85 0)
+    (property "Footprint" "Capacitor_SMD:C_0805_2012Metric_Pad1.18x1.45mm_HandSolder" (at 134.62 69.85 0)
       (effects (font (size 1.27 1.27)) hide)
     )
@@
       (effects (font (size 1.27 1.27)) (justify left))
     )
-    (property "Footprint" "" (at 78.74 44.45 0)
+    (property "Footprint" "Capacitor_SMD:C_0805_2012Metric_Pad1.18x1.45mm_HandSolder" (at 78.74 44.45 0)
       (effects (font (size 1.27 1.27)) hide)
     )
@@
       (effects (font (size 1.27 1.27)) (justify left))
     )
-    (property "Footprint" "" (at 53.34 125.73 0)
+    (property "Footprint" "Capacitor_SMD:C_0805_2012Metric_Pad1.18x1.45mm_HandSolder" (at 53.34 125.73 0)
       (effects (font (size 1.27 1.27)) hide)
     )
@@
       (effects (font (size 1.27 1.27)) (justify left))
     )
-    (property "Footprint" "" (at 140.97 113.03 0)
+    (property "Footprint" "Resistor_SMD:R_0805_2012Metric_Pad1.20x1.40mm_HandSolder" (at 140.97 113.03 0)
       (effects (font (size 1.27 1.27)) hide)
     )
@@
       (effects (font (size 1.27 1.27)) (justify left))
     )
-    (property "Footprint" "" (at 133.35 50.8 0)
+    (property "Footprint" "Capacitor_SMD:C_0805_2012Metric_Pad1.18x1.45mm_HandSolder" (at 133.35 50.8 0)
       (effects (font (size 1.27 1.27)) hide)
     )
@@
       (effects (font (size 1.27 1.27)) (justify left))
     )
-    (property "Footprint" "" (at 140.97 139.7 0)
+    (property "Footprint" "Resistor_SMD:R_0805_2012Metric_Pad1.20x1.40mm_HandSolder" (at 140.97 139.7 0)
       (effects (font (size 1.27 1.27)) hide)
     )
@@
       (effects (font (size 1.27 1.27)) (justify left))
     )
-    (property "Footprint" "" (at 38.1 119.38 0)
+    (property "Footprint" "Resistor_SMD:R_0805_2012Metric_Pad1.20x1.40mm_HandSolder" (at 38.1 119.38 0)
       (effects (font (size 1.27 1.27)) hide)
     )
@@
       (effects (font (size 1.27 1.27)) (justify left))
     )
-    (property "Footprint" "" (at 41.91 54.61 0)
+    (property "Footprint" "Capacitor_SMD:C_0805_2012Metric_Pad1.18x1.45mm_HandSolder" (at 41.91 54.61 0)
       (effects (font (size 1.27 1.27)) hide)
     )
@@
       (effects (font (size 1.27 1.27)) (justify left))
     )
-    (property "Footprint" "" (at 58.42 44.45 0)
-      (effects (font (size 1.27 1.27)) hide)
-    )
+    (property "Footprint" "Capacitor_SMD:C_0805_2012Metric_Pad1.18x1.45mm_HandSolder" (at 58.42 44.45 0)
+      (effects (font (size 1.27 1.27)) hide)
+    )
