File: PCB/servo_cpu/input-output.kicad_sch (KiCad schematic)
At the start: 1 part, among them J8 IO

Commit message: cpu pcb
Parts:
- added C2 (x2): 100n, symbol Device:C_Small
- added D3 (x2): BZT52B5v1, Diode_SMD:D_SOD-123F, symbol Diode:BZT52Bxx
- added JP2: OPA-V, Jumper:SolderJumper-3_P1.3mm_Bridged12_Pad1.0x1.5mm, symbol Jumper:SolderJumper_3_Bridged12
- added R6 (x2): 150R, symbol Device:R_Small
- added R6 (x4): 10k, symbol Device:R_Small
- added R6 (x4): 3k3, symbol Device:R_Small
- added U12: TS912, symbol Amplifier_Operational:TS912
- J8: value IO -> I/O
Connections:
- net AIN1: now reaches J8.1 (Pin_1)
- net AIN1: now also R6.2
- net +5V: now reaches J8.2 (Pin_2)
- net +5V: now also R6.2, R6.2, U12.8 (V+)
- net AIN2: now reaches J8.3 (Pin_3)
- net AIN2: now also R6.2
- net -5V: now reaches J8.4 (Pin_4)
- net -5V: now also JP2.3 (B)
- net GNDA: now reaches J8.5 (Pin_5)
- net GNDA: now also J8.6 (Pin_6), C2.2, C2.2, D3.2 (A), D3.2 (A), JP2.2 (C), R6.1, R6.1, R6.1, R6.1
- new net: C2.1, D3.1 (K), R6.1, R6.1, R6.2, R6.2, U12.3 (+)
- new net: R6.2, U12.6 (-), U12.7
- new net: JP2.1 (A), U12.4 (V-)
- new net: R6.2, U12.1, U12.2 (-)
- new net: C2.1, D3.1 (K), R6.1, R6.1, R6.2, R6.2, U12.5 (+)
- new net AIN1_ADC: R6.1
- new net AIN2_ADC: R6.1

Commit message: CPU schematic done
Parts:
- added C2 (x4): 100n, symbol Device:C_Small
- added D14: 1N4148, Diode_SMD:D_SOD-123F, symbol Device:D_Small
- added D3 (x5): BZT52B5v1, Diode_SMD:D_SOD-123F, symbol Diode:BZT52Bxx
- added R6 (x10): 10k, symbol Device:R_Small
- added R6 (x7): 2k2, symbol Device:R_Small
- added R6 (x2): 1k, symbol Device:R_Small
- added R6 (x2): 470R, symbol Device:R_Small
- added U13: 74HC14, symbol 74xx:74HC14
- added U14, U15: ~, Package_SO:SOIC-8_3.9x4.9mm_P1.27mm, symbol isp742ri:ISP742
- added U16: TS912, symbol Amplifier_Operational:TS912
- added U17: VO0661T, Package_SO:SOIC-8_3.9x4.9mm_P1.27mm, symbol Isolator:VO0661T
- added U18: 74LVC2G04, symbol 74xGxx:74LVC2G04
Connections:
- net +5V: now also J8.1 (Pin_1), C2.1, C2.1, C2.1, C2.1, R6.2, R6.2, U13.14 (VCC), U17.8 (VCC), U18.5 (VCC); no longer J8.2 (Pin_2)
- net -5V: now also J8.3 (Pin_3); no longer J8.4 (Pin_4)
- net AIN1: now also J8.5 (Pin_5); no longer J8.1 (Pin_1)
- net AIN2: now also J8.6 (Pin_6); no longer J8.3 (Pin_3)
- net GNDA: now also J8.2 (Pin_2); no longer J8.5 (Pin_5), J8.6 (Pin_6)
- net DIN4: now reaches J8.10 (Pin_10)
- net DIN4: now also R6.2
- net DIN5: now reaches J8.11 (Pin_11)
- net DIN5: now also R6.2
- net DOUT1: now reaches J8.12 (Pin_12)
- net DOUT1: now also U14.3 (OUT)
- net DOUT2: now reaches J8.13 (Pin_13)
- net DOUT2: now also U15.3 (OUT)
- net AOUT1: now reaches J8.14 (Pin_14)
- net AOUT1: now also U16.1, U16.2 (-)
- net AOUT2: now reaches J8.15 (Pin_15)
- net AOUT2: now also U16.6 (-), U16.7
- net STEP_F: now reaches J8.16 (Pin_16)
- net STEP_F: now also R6.1
- net STEP_R: now reaches J8.17 (Pin_17)
- net STEP_R: now also R6.1
- net STEP_COMM: now reaches J8.18 (Pin_18)
- net STEP_COMM: now also R6.1, R6.2, U17.2 (C1), U17.3 (C2)
- net A_OUT: now reaches J8.19 (Pin_19)
- net A_OUT: now also U18.6
- net B_OUT: now reaches J8.20 (Pin_20)
- net B_OUT: now also U18.4
- net DIN1: now reaches J8.7 (Pin_7)
- net DIN1: now also R6.2
- net DIN2: now reaches J8.8 (Pin_8)
- net DIN2: now also R6.2
- net DIN3: now reaches J8.9 (Pin_9)
- net DIN3: now also R6.2
- net at JP2.1 (A), U12.4 (V-): now also C2.2
- new net: R6.1, U13.2
- new net: D3.1 (K), R6.1, R6.2, U13.5
- new net: R6.1, U13.6
- new net: D3.1 (K), R6.1, R6.2, U13.3
- new net: R6.1, U13.4
- new net: D3.1 (K), R6.1, R6.2, U13.9
- new net: D14.1 (K), J8.4 (Pin_4)
- new net: D3.1 (K), R6.1, R6.2, U13.1
- new net: D3.1 (K), R6.1, R6.2, U13.11
- new net: R6.1, R6.2, U17.4 (A2)
- new net: R6.2, R6.2, U17.1 (A1)
- new net: R6.1, U13.10
- new net: R6.1, U13.8
- new net +24V: D14.2 (A), U14.5 (Vbb), U14.6 (Vbb), U14.7 (Vbb), U14.8 (Vbb), U15.5 (Vbb), U15.6 (Vbb), U15.7 (Vbb), U15.8 (Vbb)
- new net DAC1: U16.3 (+)
- new net DAC2: U16.5 (+)
- new net DIN1_CPU: R6.2
- new net DIN2_CPU: R6.2
- new net DIN3_CPU: R6.2
- new net DIN4_CPU: R6.2
- new net DIN5_CPU: R6.2
- new net DOUT1_CPU: U14.2 (IN)
- new net DOUT1_STATUS: U14.4 (ST)
- new net DOUT2_CPU: U15.2 (IN)
- new net DOUT2_STATUS: U15.4 (ST)
- new net ENC_A_OUT_CPU: U18.1
- new net ENC_B_OUT_CPU: U18.3
- new net GND: C2.2, C2.2, C2.2, D3.2 (A), D3.2 (A), D3.2 (A), D3.2 (A), D3.2 (A), R6.1, R6.1, R6.1, R6.1, R6.1, U13.13, U13.7 (GND), U14.1 (GND), U15.1 (GND), U17.5 (GND), U18.2 (GND)
- new net STEP_F_CPU: R6.1, U17.7 (VO1)
- new net STEP_R_CPU: R6.1, U17.6 (VO2)
- no-connect marks 0 -> 1
Other:
- note added: "ANALOG IN"
- note added: "ANALOG OUT"
- note added: "DIGITAL IN"
- note added: "DIGITAL OUT"
- note added: "ENCODER OUT"
- note added: "I/O connector"
- note added: "STEP/DIR INPUT"
- title: (none) -> External I/O
- moved on the sheet: J8, JP2, U12C

Commit message: cpu pcb layout
Parts:
- C2: footprint (none) -> Capacitor_SMD:C_0805_2012Metric_Pad1.18x1.45mm_HandSolder
- R6: footprint (none) -> Resistor_SMD:R_0805_2012Metric_Pad1.20x1.40mm_HandSolder
- U12, U16: footprint (none) -> Package_SO:SO-8_3.9x4.9mm_P1.27mm
- U13: footprint (none) -> Package_SO:SO-14_3.9x8.65mm_P1.27mm
- U14, U15: value ~ -> ISP742RI
- U18: footprint (none) -> Package_SO:SC-74-6_1.5x2.9mm_P0.95mm
Connections:
- net +5V: now also U16.8 (V+)
- net GNDA: now also U16.4 (V-)
