File: PCB/servo_cpu/power.kicad_sch (KiCad schematic)
At the start: 7 parts, among them U4 AP1117-33, U5 MC34063AD

Commit message: cpu pcb
Parts:
- removed U5: MC34063AD, Package_SO:SOIC-8_3.9x4.9mm_P1.27mm, symbol Regulator_Switching:MC34063AD
- added C27: 100n, symbol Device:C_Small
- added C28, C29, C30: 22u, Capacitor_SMD:C_0805_2012Metric_Pad1.18x1.45mm_HandSolder, symbol Device:C_Small
- added C31: 22u, symbol Device:C_Small
- added D1: SM6T27A, Diode_SMD:D_SMB, symbol Diode:SM6T27A
- added D2: US1B, Diode_SMD:D_SMA, symbol Diode:US1B
- added F1: 615mA PTC, Fuse:Fuse_1206_3216Metric, symbol Device:Fuse
- added J2: Control power, TerminalBlock_RND:TerminalBlock_RND_205-00232_1x02_P5.08mm_Horizontal, symbol Connector:Screw_Terminal_01x02
- added L1: 4u7, Inductor_SMD:L_Sunlord_SWPA8040S, symbol Device:L_Small
- added L2: 10u, Inductor_SMD:L_Sunlord_SWPA5040S, symbol Device:L_Small
- added R7: 220k, symbol Device:R_Small
- added R8: 18k, symbol Device:R_Small
- added U6: AP63205WU, Package_TO_SOT_SMD:TSOT-23-6, symbol Regulator_Switching:AP63205WU
Connections:
- net GND: now also C28.2, C29.2, C30.2, C31.2, D1.2 (A2), J2.1 (Pin_1), R8.2, U6.4 (GND)
- net +5V: now reaches C2.1, U4.3 (VI)
- net +5V: now also C28.1, C29.1, C30.1, L1.2, U6.1 (FB)
- new net: C27.1, L1.1, U6.5 (SW)
- new net: R7.2, R8.1, U6.2 (EN)
- new net: C27.2, U6.6 (BST)
- new net: F1.1, J2.2 (Pin_2)
- new net: D2.2 (A), F1.2
- new net: D1.1 (A1), D2.1 (K), L2.1
- new net +24V: C31.1, L2.2, R7.1, U6.3 (IN)
Other:
- note added: "13-14V UVLO"
- note added: "Power input and 24->5v"

Commit message: cpu pcb
Parts:
- added C2: 2u2, symbol Device:C_Small
- added C39, C41: 22u, Capacitor_SMD:C_0805_2012Metric_Pad1.18x1.45mm_HandSolder, symbol Device:C_Small
- added U11: LMC7660, Package_SO:SOIC-8_3.9x4.9mm_P1.27mm, symbol Regulator_SwitchedCapacitor:LMC7660
Connections:
- net +5V: now also C2.1, U11.8 (V+)
- net GND: now also C2.2, C41.2, U11.3 (GND)
- new net: C39.1, U11.2 (CAP+)
- new net: C39.2, U11.4 (CAP-)
- new net -5V: C41.1, U11.5 (VOUT)
- no-connect marks 0 -> 2

Commit message: CPU schematic done
Other:
- note added: "Negative -5V generator"
- title: (none) -> Power
Changed lines of the file:
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@@
 (kicad_sch (version 20230121) (generator eeschema)
   (paper "A4")
+  (title_block
+    (title "Power")
+    (date "2023-03-06")
+    (rev "1")
+    (comment 1 "W. Burdecki 2023")
+    (comment 2 "github.com/wiciu15")
+  )
   (junction (at 251.46 71.12) (diameter 0) (color 0 0 0 0)
   )
@@
     (effects (font (size 1.27 1.27)) (justify left bottom))
   )
+  (text "Negative -5V generator" (at 127 127 0)
+    (effects (font (size 3 3)) (justify left bottom))
+  )
   (text "5v -> 3.3V regulator" (at 231.14 21.59 0)

Commit message: cpu pcb layout
Parts:
- added JP3: GND, Jumper:SolderJumper-2_P1.3mm_Bridged_RoundedPad1.0x1.5mm, symbol Jumper:Jumper_2_Bridged
- C2, C27, C31: footprint (none) -> Capacitor_SMD:C_0805_2012Metric_Pad1.18x1.45mm_HandSolder
- R7, R8: footprint (none) -> Resistor_SMD:R_0805_2012Metric_Pad1.20x1.40mm_HandSolder
Connections:
- net GND: now also JP3.1 (A)
- net GNDA: now also JP3.2 (B)
Changed lines of the file:
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@@
+    (stroke (width 0) (type default))
+  )
+  (wire (pts (xy 232.41 95.25) (xy 234.95 95.25))
     (stroke (width 0) (type default))
   )
@@
   )
   (wire (pts (xy 251.46 71.12) (xy 251.46 72.39))
+    (stroke (width 0) (type default))
+  )
+  (wire (pts (xy 245.11 95.25) (xy 247.65 95.25))
     (stroke (width 0) (type default))
   )
@@
       (effects (font (size 1.27 1.27)) (justify left))
     )
-    (property "Footprint" "" (at 73.66 66.04 0)
+    (property "Footprint" "Resistor_SMD:R_0805_2012Metric_Pad1.20x1.40mm_HandSolder" (at 73.66 66.04 0)
       (effects (font (size 1.27 1.27)) hide)
     )
@@
       (effects (font (size 1.27 1.27)) (justify left))
     )
-    (property "Footprint" "" (at 260.35 35.56 0)
+    (property "Footprint" "Capacitor_SMD:C_0805_2012Metric_Pad1.18x1.45mm_HandSolder" (at 260.35 35.56 0)
       (effects (font (size 1.27 1.27)) hide)
     )
@@
     )
   )
+  (symbol (lib_id "power:GND") (at 232.41 95.25 0) (unit 1)
+    (in_bom yes) (on_board yes) (dnp no)
+    (property "Reference" "#PWR03" (at 232.41 101.6 0)
+      (effects (font (size 1.27 1.27)) hide)
+    )
+    (property "Value" "GND" (at 236.22 99.06 0)
+      (effects (font (size 1.27 1.27)))
+    )
+    (property "Footprint" "" (at 232.41 95.25 0)
+      (effects (font (size 1.27 1.27)) hide)
+    )
+    (property "Datasheet" "" (at 232.41 95.25 0)
+      (effects (font (size 1.27 1.27)) hide)
+    )
+    (pin "1")
+    (instances
+      (project "servo_cpu"
+        (path "/db89e46c-646b-4fdd-b861-e9de706ced13/efadaaf3-3aa9-4d56-8b34-2b9a8a5957ea"
+          (reference "#PWR03") (unit 1)
+        )
+        (path "/db89e46c-646b-4fdd-b861-e9de706ced13"
+          (reference "#PWR022") (unit 1)
+        )
+        (path "/db89e46c-646b-4fdd-b861-e9de706ced13/731cc340-9654-433e-bcf1-701f3d0fb633"
+          (reference "#PWR0153") (unit 1)
+        )
+      )
+    )
+  )
   (symbol (lib_id "power:GND") (at 167.64 146.05 0) (unit 1)
     (in_bom yes) (on_board yes) (dnp no)
@@
     )
   )
+  (symbol (lib_id "power:GNDA") (at 247.65 95.25 0) (unit 1)
+    (in_bom yes) (on_board yes) (dnp no) (fields_autoplaced)
+    (property "Reference" "#PWR023" (at 247.65 101.6 0)
+      (effects (font (size 1.27 1.27)) hide)
+    )
+    (property "Value" "GNDA" (at 247.65 100.33 0)
+      (effects (font (size 1.27 1.27)))
+    )
+    (property "Footprint" "" (at 247.65 95.25 0)
+      (effects (font (size 1.27 1.27)) hide)
+    )
+    (property "Datasheet" "" (at 247.65 95.25 0)
+      (effects (font (size 1.27 1.27)) hide)
+    )
+    (pin "1")
+    (instances
+      (project "servo_cpu"
+        (path "/db89e46c-646b-4fdd-b861-e9de706ced13"
+          (reference "#PWR023") (unit 1)
+        )
+        (path "/db89e46c-646b-4fdd-b861-e9de706ced13/731cc340-9654-433e-bcf1-701f3d0fb633"
+          (reference "#PWR0152") (unit 1)
+        )
+      )
+    )
+  )
   (symbol (lib_id "power:+5V") (at 118.11 140.97 0) (unit 1)
     (in_bom yes) (on_board yes) (dnp no) (fields_autoplaced)
@@
     )
   )
+  (symbol (lib_id "Jumper:Jumper_2_Bridged") (at 240.03 95.25 0) (unit 1)
+    (in_bom yes) (on_board yes) (dnp no) (fields_autoplaced)
+    (property "Reference" "JP3" (at 240.03 90.17 0)
+      (effects (font (size 1.27 1.27)))
+    )
+    (property "Value" "GND" (at 240.03 92.71 0)
+      (effects (font (size 1.27 1.27)))
+    )
+    (property "Footprint" "Jumper:SolderJumper-2_P1.3mm_Bridged_RoundedPad1.0x1.5mm" (at 240.03 95.25 0)
+      (effects (font (size 1.27 1.27)) hide)
+    )
+    (property "Datasheet" "~" (at 240.03 95.25 0)
+      (effects (font (size 1.27 1.27)) hide)
+    )
+    (pin "1")
+    (pin "2")
+    (instances
+      (project "servo_cpu"
+        (path "/db89e46c-646b-4fdd-b861-e9de706ced13/731cc340-9654-433e-bcf1-701f3d0fb633"
+          (reference "JP3") (unit 1)
+        )
+      )
+    )
+  )
   (symbol (lib_id "power:+3.3VA") (at 251.46 71.12 0) (unit 1)
     (in_bom yes) (on_board yes) (dnp no) (fields_autoplaced)
@@
       (effects (font (size 1.27 1.27)) (justify left))
     )
-    (property "Footprint" "" (at 251.46 74.93 0)
+    (property "Footprint" "Capacitor_SMD:C_0805_2012Metric_Pad1.18x1.45mm_HandSolder" (at 251.46 74.93 0)
       (effects (font (size 1.27 1.27)) hide)
     )
@@
       (effects (font (size 1.27 1.27)) (justify left))
     )
-    (property "Footprint" "" (at 73.66 71.12 0)
+    (property "Footprint" "Resistor_SMD:R_0805_2012Metric_Pad1.20x1.40mm_HandSolder" (at 73.66 71.12 0)
       (effects (font (size 1.27 1.27)) hide)
     )
@@
       (effects (font (size 1.27 1.27)) (justify left))
     )
-    (property "Footprint" "" (at 118.11 143.51 0)
+    (property "Footprint" "Capacitor_SMD:C_0805_2012Metric_Pad1.18x1.45mm_HandSolder" (at 118.11 143.51 0)
       (effects (font (size 1.27 1.27)) hide)
     )
@@
         )
         (path "/db89e46c-646b-4fdd-b861-e9de706ced13/731cc340-9654-433e-bcf1-701f3d0fb633"
-          (reference "22u1") (unit 1)
+          (reference "L3") (unit 1)
         )
       )
@@
       (effects (font (size 1.27 1.27)) (justify left))
     )
-    (property "Footprint" "" (at 234.95 35.56 0)
+    (property "Footprint" "Capacitor_SMD:C_0805_2012Metric_Pad1.18x1.45mm_HandSolder" (at 234.95 35.56 0)
       (effects (font (size 1.27 1.27)) hide)
     )
@@
       (effects (font (size 1.27 1.27)) (justify left))
     )
-    (property "Footprint" "" (at 64.77 66.04 0)
+    (property "Footprint" "Capacitor_SMD:C_0805_2012Metric_Pad1.18x1.45mm_HandSolder" (at 64.77 66.04 0)
       (effects (font (size 1.27 1.27)) hide)
     )
@@
       (effects (font (size 1.27 1.27)) (justify left))
     )
-    (property "Footprint" "" (at 114.3 66.04 0)
+    (property "Footprint" "Capacitor_SMD:C_0805_2012Metric_Pad1.18x1.45mm_HandSolder" (at 114.3 66.04 0)
       (effects (font (size 1.27 1.27)) hide)
     )
@@
       (effects (font (size 1.27 1.27)) (justify left))
     )
-    (property "Footprint" "" (at 241.3 74.93 0)
-      (effects (font (size 1.27 1.27)) hide)
-    )
+    (property "Footprint" "Capacitor_SMD:C_0805_2012Metric_Pad1.18x1.45mm_HandSolder" (at 241.3 74.93 0)
+      (effects (font (size 1.27 1.27)) hide)
+    )
