File: PCB/servo_cpu/servo_cpu.kicad_sch (KiCad schematic)
At the start: 24 parts, among them J1 PWR board, U1 STM32F407VETx, U3 TS912, Y1 16M xt224

Commit message: cpu pcb
Parts:
- added J6: DEBUG, symbol Connector_Generic:Conn_01x04
Connections:
- net +3V3: now also J6.4 (Pin_4)
- net GND: now also J6.1 (Pin_1)
- net /ENCODER_SHORT: now reaches U1.34 (PC5)
- net BTN_ENTER: now reaches U1.55 (PD8)
- net BTN_UP: now reaches U1.56 (PD9)
- net BTN_DOWN: now reaches U1.57 (PD10)
- net BTN_ESC: now reaches U1.58 (PD11)
- net LED_STATUS: now reaches U1.61 (PD14)
- net LED_ERROR: now reaches U1.62 (PD15)
- net ENC_A: now reaches U1.63 (PC6)
- net ENC_B: now reaches U1.64 (PC7)
- net ENC_Z: now reaches U1.65 (PC8)
- net ENCODER_ENABLE: now reaches U1.66 (PC9)
- net ENCODER_DE: now reaches U1.67 (PA8)
- net ENCODER_TX: now reaches U1.68 (PA9)
- net ENCODER_RX: now reaches U1.69 (PA10)
- net USB_N: now reaches U1.70 (PA11)
- net USB_P: now reaches U1.71 (PA12)
- net DEBUG_IO: now reaches U1.72 (PA13)
- net DEBUG_IO: now also J6.2 (Pin_2)
- net DEBUG_CLK: now reaches U1.76 (PA14)
- net DEBUG_CLK: now also J6.3 (Pin_3)
- net CAN_RX: now reaches U1.81 (PD0)
- net CAN_TX: now reaches U1.82 (PD1)
- net MODBUS_TX: now reaches U1.86 (PD5)
- net MODBUS_RX: now reaches U1.87 (PD6)
- net MODBUS_DE: now reaches U1.96 (PB9)
Other:
- added sheet Connectivity (connectivity.kicad_sch)
- added sheet Encoder (encoder.kicad_sch)

Commit message: cpu schematic
Other:
- added sheet input-output (input-output.kicad_sch)
Changed lines of the file:
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@@
+    )
+  )
+  (sheet (at 259.08 54.61) (size 21.59 11.43) (fields_autoplaced)
+    (stroke (width 0.1524) (type solid))
+    (fill (color 0 0 0 0.0000))
+    (property "Sheetname" "input-output" (at 259.08 53.8984 0)
+      (effects (font (size 1.27 1.27)) (justify left bottom))
+    )
+    (property "Sheetfile" "input-output.kicad_sch" (at 259.08 66.6246 0)
+      (effects (font (size 1.27 1.27)) (justify left top))
+    )
+    (instances
+      (project "servo_cpu"
+        (path "/db89e46c-646b-4fdd-b861-e9de706ced13" (page "7"))
+      )
     )
   )

Commit message: CPU schematic done
Connections:
- net MODBUS_DE: now also U1.88 (PD7)
- net DIN3_CPU: now reaches U1.1 (PE2)
- net DOUT1_STATUS: now reaches U1.15 (PC0)
- net DOUT2_STATUS: now reaches U1.16 (PC1)
- net DIN4_CPU: now reaches U1.2 (PE3)
- net AIN1_ADC: now reaches U1.25 (PA2)
- net AIN2_ADC: now reaches U1.26 (PA3)
- net DAC1: now reaches U1.29 (PA4)
- net DIN5_CPU: now reaches U1.3 (PE4)
- net DAC2: now reaches U1.30 (PA5)
- net DOUT1_CPU: now reaches U1.4 (PE5)
- net DOUT2_CPU: now reaches U1.5 (PE6)
- net ENC_A_OUT_CPU: now reaches U1.51 (PB12)
- net ENC_B_OUT_CPU: now reaches U1.52 (PB13)
- net STEP_F_CPU: now reaches U1.59 (PD12)
- net STEP_R_CPU: now reaches U1.60 (PD13)
- net EXT_CLK: now reaches U1.78 (PC10)
- net EXT_MISO: now reaches U1.79 (PC11)
- net EXT_MOSI: now reaches U1.80 (PC12)
- net EXT_INT: now reaches U1.83 (PD2)
- net EXT_RESET: now reaches U1.84 (PD3)
- net EXT_CS: now reaches U1.85 (PD4)
- net DIN1_CPU: now reaches U1.97 (PE0)
- net DIN2_CPU: now reaches U1.98 (PE1)
- no-connect marks 1 -> 13
Other:
- title: (none) -> Servo2 CPU board

Commit message: cpu pcb layout
Parts:
- C2: footprint (none) -> Capacitor_SMD:C_0805_2012Metric_Pad1.18x1.45mm_HandSolder
- J1: footprint (none) -> Connector_PinHeader_2.54mm:PinHeader_2x10_P2.54mm_Vertical
- J6: footprint (none) -> Connector_PinHeader_2.54mm:PinHeader_1x04_P2.54mm_Vertical
- R4, R5, R6: footprint (none) -> Resistor_SMD:R_0805_2012Metric_Pad1.20x1.40mm_HandSolder
- U3: footprint (none) -> Package_SO:SO-8_3.9x4.9mm_P1.27mm
Changed lines of the file:
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@@
       (effects (font (size 1.27 1.27)) (justify left))
     )
-    (property "Footprint" "" (at 46.99 152.4 0)
+    (property "Footprint" "Capacitor_SMD:C_0805_2012Metric_Pad1.18x1.45mm_HandSolder" (at 46.99 152.4 0)
       (effects (font (size 1.27 1.27)) hide)
     )
@@
       (effects (font (size 1.27 1.27)))
     )
-    (property "Footprint" "" (at 156.21 50.8 0)
+    (property "Footprint" "Package_SO:SO-8_3.9x4.9mm_P1.27mm" (at 156.21 50.8 0)
       (effects (font (size 1.27 1.27)) hide)
     )
@@
       (effects (font (size 1.27 1.27)) (justify left))
     )
-    (property "Footprint" "" (at 95.25 20.32 0)
+    (property "Footprint" "Capacitor_SMD:C_0805_2012Metric_Pad1.18x1.45mm_HandSolder" (at 95.25 20.32 0)
       (effects (font (size 1.27 1.27)) hide)
     )
@@
       (effects (font (size 1.27 1.27)) (justify left))
     )
-    (property "Footprint" "" (at 139.7 20.32 0)
+    (property "Footprint" "Capacitor_SMD:C_0805_2012Metric_Pad1.18x1.45mm_HandSolder" (at 139.7 20.32 0)
       (effects (font (size 1.27 1.27)) hide)
     )
@@
       (effects (font (size 1.27 1.27)) (justify left))
     )
-    (property "Footprint" "" (at 16.51 48.26 0)
+    (property "Footprint" "Capacitor_SMD:C_0805_2012Metric_Pad1.18x1.45mm_HandSolder" (at 16.51 48.26 0)
       (effects (font (size 1.27 1.27)) hide)
     )
@@
       (effects (font (size 1.27 1.27)) (justify left))
     )
-    (property "Footprint" "" (at 104.14 20.32 0)
+    (property "Footprint" "Capacitor_SMD:C_0805_2012Metric_Pad1.18x1.45mm_HandSolder" (at 104.14 20.32 0)
       (effects (font (size 1.27 1.27)) hide)
     )
@@
       (effects (font (size 1.27 1.27)) (justify left))
     )
-    (property "Footprint" "" (at 157.48 33.02 0)
+    (property "Footprint" "Package_SO:SO-8_3.9x4.9mm_P1.27mm" (at 157.48 33.02 0)
       (effects (font (size 1.27 1.27)) hide)
     )
@@
       (effects (font (size 1.27 1.27)) (justify left))
     )
-    (property "Footprint" "" (at 130.81 20.32 0)
+    (property "Footprint" "Capacitor_SMD:C_0805_2012Metric_Pad1.18x1.45mm_HandSolder" (at 130.81 20.32 0)
       (effects (font (size 1.27 1.27)) hide)
     )
@@
       (effects (font (size 1.27 1.27)) (justify left))
     )
-    (property "Footprint" "" (at 33.02 68.58 0)
+    (property "Footprint" "Capacitor_SMD:C_0805_2012Metric_Pad1.18x1.45mm_HandSolder" (at 33.02 68.58 0)
       (effects (font (size 1.27 1.27)) hide)
     )
@@
       (effects (font (size 1.27 1.27)) (justify left))
     )
-    (property "Footprint" "" (at 172.72 68.58 0)
+    (property "Footprint" "Capacitor_SMD:C_0805_2012Metric_Pad1.18x1.45mm_HandSolder" (at 172.72 68.58 0)
       (effects (font (size 1.27 1.27)) hide)
     )
@@
       (effects (font (size 1.27 1.27)) (justify left))
     )
-    (property "Footprint" "" (at 121.92 20.32 0)
+    (property "Footprint" "Capacitor_SMD:C_0805_2012Metric_Pad1.18x1.45mm_HandSolder" (at 121.92 20.32 0)
       (effects (font (size 1.27 1.27)) hide)
     )
@@
       (effects (font (size 1.27 1.27)))
     )
-    (property "Footprint" "" (at 175.26 66.04 0)
+    (property "Footprint" "Resistor_SMD:R_0805_2012Metric_Pad1.20x1.40mm_HandSolder" (at 175.26 66.04 0)
       (effects (font (size 1.27 1.27)) hide)
     )
@@
       (effects (font (size 1.27 1.27)) (justify left))
     )
-    (property "Footprint" "" (at 172.72 50.8 0)
+    (property "Footprint" "Capacitor_SMD:C_0805_2012Metric_Pad1.18x1.45mm_HandSolder" (at 172.72 50.8 0)
       (effects (font (size 1.27 1.27)) hide)
     )
@@
       (effects (font (size 1.27 1.27)) (justify left))
     )
-    (property "Footprint" "" (at 24.13 68.58 0)
+    (property "Footprint" "Capacitor_SMD:C_0805_2012Metric_Pad1.18x1.45mm_HandSolder" (at 24.13 68.58 0)
       (effects (font (size 1.27 1.27)) hide)
     )
@@
       (effects (font (size 1.27 1.27)))
     )
-    (property "Footprint" "" (at 247.65 142.24 0)
+    (property "Footprint" "Connector_PinHeader_2.54mm:PinHeader_2x10_P2.54mm_Vertical" (at 247.65 142.24 0)
       (effects (font (size 1.27 1.27)) hide)
     )
@@
       (effects (font (size 1.27 1.27)) (justify left))
     )
-    (property "Footprint" "" (at 36.83 149.86 0)
+    (property "Footprint" "Capacitor_SMD:C_0805_2012Metric_Pad1.18x1.45mm_HandSolder" (at 36.83 149.86 0)
       (effects (font (size 1.27 1.27)) hide)
     )
@@
       (effects (font (size 1.27 1.27)) (justify left))
     )
-    (property "Footprint" "" (at 113.03 20.32 0)
+    (property "Footprint" "Capacitor_SMD:C_0805_2012Metric_Pad1.18x1.45mm_HandSolder" (at 113.03 20.32 0)
       (effects (font (size 1.27 1.27)) hide)
     )
@@
       (effects (font (size 1.27 1.27)) (justify left))
     )
-    (property "Footprint" "" (at 110.49 29.21 0)
+    (property "Footprint" "Capacitor_SMD:C_0805_2012Metric_Pad1.18x1.45mm_HandSolder" (at 110.49 29.21 0)
       (effects (font (size 1.27 1.27)) hide)
     )
@@
       (effects (font (size 1.27 1.27)))
     )
-    (property "Footprint" "" (at 27.94 38.1 0)
+    (property "Footprint" "Resistor_SMD:R_0805_2012Metric_Pad1.20x1.40mm_HandSolder" (at 27.94 38.1 0)
       (effects (font (size 1.27 1.27)) hide)
     )
@@
       (effects (font (size 1.27 1.27)) (justify left))
     )
-    (property "Footprint" "" (at 27.94 25.4 0)
+    (property "Footprint" "Capacitor_SMD:C_0805_2012Metric_Pad1.18x1.45mm_HandSolder" (at 27.94 25.4 0)
       (effects (font (size 1.27 1.27)) hide)
     )
@@
       (effects (font (size 1.27 1.27)))
     )
-    (property "Footprint" "" (at 175.26 48.26 0)
+    (property "Footprint" "Resistor_SMD:R_0805_2012Metric_Pad1.20x1.40mm_HandSolder" (at 175.26 48.26 0)
       (effects (font (size 1.27 1.27)) hide)
     )
@@
       (effects (font (size 1.27 1.27)) (justify left))
     )
-    (property "Footprint" "" (at 168.91 31.75 0)
+    (property "Footprint" "Capacitor_SMD:C_0805_2012Metric_Pad1.18x1.45mm_HandSolder" (at 168.91 31.75 0)
       (effects (font (size 1.27 1.27)) hide)
     )
@@
       (effects (font (size 1.27 1.27)) (justify left))
     )
-    (property "Footprint" "" (at 257.81 95.25 0)
+    (property "Footprint" "Connector_PinHeader_2.54mm:PinHeader_1x04_P2.54mm_Vertical" (at 257.81 95.25 0)
       (effects (font (size 1.27 1.27)) hide)
     )
@@
       (effects (font (size 1.27 1.27)))
     )
-    (property "Footprint" "" (at 156.21 68.58 0)
-      (effects (font (size 1.27 1.27)) hide)
-    )
+    (property "Footprint" "Package_SO:SO-8_3.9x4.9mm_P1.27mm" (at 156.21 68.58 0)
+      (effects (font (size 1.27 1.27)) hide)
+    )

Commit message: cpu pcb routing
Connections:
- net MODBUS_DE: no longer U1.96 (PB9)
- no-connect marks 13 -> 14
Changed lines of the file:
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@@
   (no_connect (at 107.95 116.84))
   (no_connect (at 107.95 157.48))
+  (no_connect (at 107.95 104.14))
   (no_connect (at 62.23 99.06))
   (no_connect (at 62.23 91.44))
@@
       (effects (font (size 1.27 1.27)) (justify left) hide)
     )
-  )
-  (global_label "MODBUS_DE" (shape input) (at 107.95 104.14 0) (fields_autoplaced)
-    (effects (font (size 1.27 1.27)) (justify left))
-    (property "Intersheetrefs" "${INTERSHEET_REFS}" (at 122.1043 104.14 0)
-      (effects (font (size 1.27 1.27)) (justify left) hide)
-    )
