File: PCB/servo_cpu/servo_cpu.kicad_pcb (KiCad board)
At the start: 4 copper layers, 96 x 172 mm, 166 parts, among them J1 PWR board, J2 Control power, J3 ABZ, J4 Serial Encoder, J5 CONN, J6 DEBUG, J7 USB_B, J8 I/O, J9 EXT, SW1 ENTER, SW2 ESC, SW3 UP, SW4 DOWN, U1 STM32F407VETx, U10 SN65HVD232, U11 LMC7660, U12 TS912, U13 74HC14, U14 ISP742RI, U15 ISP742RI, U16 TS912, U17 VO0661T, U18 74LVC2G04, U2 M24C02-WMN, U3 TS912, U4 AP1117-33, U5 ISL83491, U6 AP63205WU, U7 AM26LS32A, U8 AP2151A, U9 MAX485E, Y1 16M xt224

Commit message: cpu pcb routing
Parts:
- moved C40 172.4 mm to (95.5, 170.4), turned to 180 degrees
- moved C41 168.5 mm to (95.9, 161.0)
- moved C39 166.1 mm to (101.1, 164.5), turned to 90 degrees
- moved R42 153.6 mm to (83.5, 130.4), turned to 180 degrees
- moved R43 149.2 mm to (83.5, 125.7)
- moved R46 145.6 mm to (83.5, 128.0)
- moved R47 141.8 mm to (83.5, 123.5)
- moved R33 141.4 mm to (83.4, 112.7), turned to 180 degrees
- moved R36 138.1 mm to (83.4, 115.4), turned to 180 degrees
- moved R37 138.1 mm to (83.4, 118.3)
- moved R39 136.4 mm to (83.5, 120.9), turned to 180 degrees
- moved R34 133.7 mm to (90.8, 112.9), turned to 180 degrees
- moved R17 128.8 mm to (83.4, 104.1), turned to 180 degrees
- moved R40 128.5 mm to (91.1, 121.3), turned to 180 degrees
- moved R30 127.0 mm to (83.4, 106.8), turned to 180 degrees
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Connections:
- C14 pad 2: GND -> GNDA
- U1 pad 96: MODBUS_DE -> unconnected-(U1-PB9-Pad96)
Routing:
- net +5V: track 0.00 -> 498.3 mm, vias 0 -> 23
- net GND: track 0.00 -> 416.7 mm, vias 0 -> 56
- net GNDA: track 0.00 -> 303.0 mm, vias 0 -> 14
- net +3V3: track 0.00 -> 185.4 mm, vias 0 -> 23
- net /DISPLAY_CS: track 0.00 -> 171.0 mm, vias 0 -> 2
- net +24V: track 0.00 -> 169.8 mm, vias 0 -> 6
- net /DISPLAY_RESET: track 0.00 -> 169.3 mm, vias 0 -> 2
- net -5V: track 0.00 -> 167.0 mm, vias 0 -> 8
- net DISPLAY_CLK: track 0.00 -> 166.0 mm, vias 0 -> 2
- net DISPLAY_MOSI: track 0.00 -> 159.0 mm, vias 0 -> 2
- net LED_STATUS: track 0.00 -> 157.8 mm, vias 0 -> 2
- net LED_ERROR: track 0.00 -> 155.6 mm, vias 0 -> 2
- net BTN_ESC: track 0.00 -> 140.7 mm, vias 0 -> 2
- net USB_N: track 0.00 -> 136.4 mm, vias 0 -> 3
- net USB_P: track 0.00 -> 136.2 mm, vias 0 -> 3
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- added copper zone on F.Cu, net +3V3
- added copper zone on In1.Cu, net +3V3
- added copper zone on In1.Cu, net +5V
- added copper zone on In2.Cu, net GND
Other:
- board text added: "ERROR"
- board text added: "STATUS"

Commit message: cpu board done
Parts:
- added REF**: ESD-Logo_8.9x8mm_SilkScreen, Symbol:ESD-Logo_8.9x8mm_SilkScreen, F.Cu at (83.2, 81.7)
- moved C31 1.36 mm to (94.6, 175.5)
- moved J2 0.55 mm to (88.7, 184.6)
Routing:
- net /A: track 29.3 -> 33.8 mm
- net +24V: track 169.8 -> 167.0 mm
- net +5V: track 498.3 -> 500.7 mm
- net A: track 27.7 -> 29.9 mm
- net GND: track 416.7 -> 415.2 mm
- net CANL: track 17.5 -> 16.1 mm
- net Net-(U6-SW): track 10.8 -> 9.69 mm
- net AIN1: track 17.8 -> 16.6 mm
- net MR: track 26.4 -> 25.4 mm
- net +3V3: track 185.4 -> 185.8 mm, vias 23 -> 24
Other:
- board text added: "+5"
- board text added: "-5"
- board text added: "/CS"
- board text added: "/FLT"
- board text added: "24V"
- board text added: "3v3"
- board text added: "5 G INT C RES O CS I"
- board text added: "5V"
- board text added: "A"
- board text added: "A+"
- board text added: "A-"
- board text added: "A1"
- board text added: "A2"
- board text added: "B"
- board text added: "B+"
- board text added: "B-"
- board text added: "BRK"
- board text added: "CANH"
- board text added: "CANL"
- board text added: "CANR"
- board text added: "CANT"
- board text added: "CK"
- board text added: "CLK"
- board text added: "CS"
- board text added: "D+"
- board text added: "D-"
- board text added: "DAC1"
- board text added: "DAC2"
- board text added: "DE"
- board text added: "DI"
- board text added: "G"
- board text added: "GND"
- board text added: "GNDA"
- board text added: "IO"
- board text added: "IV"
- board text added: "N"
- board text added: "P"
- board text added: "R+"
- board text added: "R-"
- board text added: "RES"
- board text added: "RX"
- board text added: "SCL"
- board text added: "SDA"
- board text added: "SS"
- board text added: "Servo2 CPU W.Burdecki 2023 github.com/wiciu15"
- board text added: "TX"
- board text added: "UH"
- board text added: "UL"
- board text added: "VL"
- board text added: "WH"
- board text added: "WL"
- board text added: "Z"
- board text added: "Z+"
- board text added: "Z-"
- board text added: "rx"
- board text added: "tx"
- board text added: "x"
